File: variable load.kicad_pcb (KiCad board)
At the start: 2 copper layers, 130.2 x 99.2 mm, 42 parts, among them IC1 OPA4197ID, IC2 OPA4197ID, J1 Screw_Terminal_01x02, J2 Screw_Terminal_01x03, J3 Screw_Terminal_01x02, Q1 IXTX110N20L2, Q2 IXTX110N20L2, Q3 IXTX110N20L2, Q4 IXTX110N20L2, Q5 IXTX110N20L2, Q6 IXTX110N20L2, Q7 IXTX110N20L2, Q8 IXTX110N20L2

Commit message: rerouted everything and included max's additions
Parts:
- added C13: 100nF, Capacitor_SMD:C_0805_2012Metric, F.Cu at (68.5, 102.0)
- added C14: 10uF, Capacitor_SMD:C_1206_3216Metric, F.Cu at (58.8, 109.0)
- added C15: 10uF, Package_SO:SOIC-8_3.9x4.9mm_P1.27mm, F.Cu at (89.0, 104.5)
- added C16: 10uF, Package_SO:SOIC-8_3.9x4.9mm_P1.27mm, F.Cu at (69.5, 96.5)
- added C17: 100nF, Capacitor_SMD:C_0805_2012Metric, F.Cu at (65.8, 102.0)
- added C18: 100nF, Capacitor_SMD:C_0805_2012Metric, F.Cu at (68.4, 107.6)
- added C19: 100nF, Capacitor_SMD:C_0805_2012Metric, F.Cu at (64.2, 107.6)
- added C20: 1u, Capacitor_SMD:C_0805_2012Metric, F.Cu at (103.0, 79.0)
- added C21: 1u, Capacitor_SMD:C_0805_2012Metric, F.Cu at (115.5, 79.0)
- added C22: 10uF, Capacitor_SMD:C_1206_3216Metric, F.Cu at (115.5, 74.5)
- added IC3: OPA4197ID, Package_SO:SOIC-14_3.9x8.7mm_P1.27mm, F.Cu at (109.5, 78.0)
- added J4: Conn_01x04, Connector_PinHeader_2.54mm:PinHeader_1x04_P2.54mm_Vertical, F.Cu at (95.0, 109.5)
- added R22: 1k, Resistor_SMD:R_0805_2012Metric, F.Cu at (79.0, 91.0)
- added R24: 1k, Resistor_SMD:R_0805_2012Metric, F.Cu at (93.5, 83.0)
- added R26: 1k, Resistor_SMD:R_0805_2012Metric, F.Cu at (80.4, 95.0)
- added R27: 10k, Resistor_SMD:R_0805_2012Metric, F.Cu at (93.4, 92.5)
- added R28: 6.98k, Resistor_SMD:R_0805_2012Metric, F.Cu at (123.5, 80.5)
- added R29: 1k, Resistor_SMD:R_0805_2012Metric, F.Cu at (120.5, 77.4)
- added U1: MCP4822-E_MS, Package_SO:MSOP-8_3x3mm_P0.65mm, F.Cu at (88.0, 96.5)
- added U2: 6N137, Package_DIP:DIP-8_W7.62mm, F.Cu at (69.5, 79.5)
- added U3: R-78HE5.0-0.3, Package_SIP:SIP3_11.6x8.5mm, F.Cu at (79.5, 102.8)
- added U7: 6N137, Package_DIP:DIP-8_W7.62mm, F.Cu at (83.2, 79.2)
- added U8: 6N137, Package_DIP:DIP-8_W7.62mm, F.Cu at (105.7, 86.7)
- moved J1 15.6 mm to (125.5, 19.3)
- moved Q1 12.2 mm to (44.0, 108.0)
- moved Q2 12.2 mm to (44.0, 87.1)
- moved Q3 12.2 mm to (44.0, 67.0)
- moved Q4 12.2 mm to (44.0, 47.0)
- moved R1 12.2 mm to (52.2, 97.1)
- moved R2 12.2 mm to (50.9, 107.7)
- moved R3 12.2 mm to (52.2, 76.2)
- moved R4 12.2 mm to (50.9, 87.2)
- moved R5 12.2 mm to (52.1, 56.1)
- moved R6 12.2 mm to (50.9, 67.2)
- moved R7 12.2 mm to (52.2, 36.1)
- moved R8 12.2 mm to (50.5, 47.2)
- moved R17 9.04 mm to (109.5, 29.5)
- moved C6 7.60 mm to (76.5, 61.0), turned to 90 degrees
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Routing:
- net 5V_LOAD: track 0.00 -> 111.1 mm
- net Net-(IC1-OUT_A): track 164.5 -> 66.0 mm, vias 0 -> 2
- net 5V_LED: track 0.00 -> 84.7 mm, vias 0 -> 1
- net Net-(IC1--IN_A): track 124.0 -> 51.4 mm, vias 0 -> 2
- net +12V: track 221.2 -> 166.8 mm, vias 4 -> 9
- net Net-(IC2--INB): track 121.6 -> 74.2 mm, vias 0 -> 2
- net SCK_K: track 0.00 -> 42.7 mm, vias 0 -> 1
- net /VREF_DAC: track 0.00 -> 41.7 mm
- net CS_L: track 0.00 -> 39.3 mm, vias 0 -> 2
- net GND: track 69.2 -> 105.7 mm, vias 28 -> 44
- net SDI_K: track 0.00 -> 32.9 mm, vias 0 -> 1
- net Net-(IC1--IN_D): track 95.4 -> 63.6 mm
- net /Vturb: track 312.5 -> 281.7 mm
- net Net-(IC2-OUTB): track 106.8 -> 82.5 mm
- net SCK_L: track 0.00 -> 23.8 mm, vias 0 -> 2
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Other:
- board size 130.2 x 99.2 mm -> 117.9 x 99.2 mm
