File: variable load.kicad_sch (KiCad schematic)
At the start: 65 parts, among them IC1 OPA4197ID, IC2 OPA4197ID, IC3 OPA4197ID, J1 Screw_Terminal_01x02, J2 Screw_Terminal_01x03, J3 Screw_Terminal_01x02, J4 Conn_01x04, Q1 IXTX110N20L2, Q2 IXTX110N20L2, Q3 IXTX110N20L2, Q4 IXTX110N20L2, Q5 IXTX110N20L2, Q6 IXTX110N20L2, Q7 IXTX110N20L2, Q8 IXTX110N20L2, U1 MCP4822-E_MS, U2 6N137, U3 R-78HE5.0-0.3, U7 6N137, U8 6N137

Commit message: rerouted everything and included max's additions
Parts:
- C13, C17, C18, C19: footprint (none) -> Capacitor_SMD:C_0805_2012Metric
- C14, C22: footprint (none) -> Capacitor_SMD:C_1206_3216Metric
- J4: footprint (none) -> Connector_PinHeader_2.54mm:PinHeader_1x04_P2.54mm_Vertical
- R22, R24, R26, R27, R28, R29: footprint (none) -> Resistor_SMD:R_0805_2012Metric
- U1: footprint MCP4822-E_MS:SOP65P490X110-8N -> Package_SO:MSOP-8_3x3mm_P0.65mm
- U3: footprint R-78HE5.0-0.3:SIP900W75P254L1200H1300Q3 -> Package_SIP:SIP3_11.6x8.5mm
Connections:
- no-connect marks 7 -> 16
Changed lines of the file:
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@@
 	)
 	(junction
+		(at 234.95 151.13)
+		(diameter 0)
+		(color 0 0 0 0)
+	)
+	(junction
 		(at 232.41 123.19)
 		(diameter 0)
@@
 	)
 	(no_connect
+		(at 204.47 130.81)
+	)
+	(no_connect
+		(at 204.47 133.35)
+	)
+	(no_connect
+		(at 173.99 118.11)
+	)
+	(no_connect
+		(at 173.99 133.35)
+	)
+	(no_connect
 		(at 49.53 137.16)
 	)
@@
 	)
 	(no_connect
+		(at 204.47 128.27)
+	)
+	(no_connect
 		(at 49.53 170.18)
 	)
 	(no_connect
+		(at 173.99 123.19)
+	)
+	(no_connect
+		(at 173.99 128.27)
+	)
+	(no_connect
 		(at 49.53 147.32)
 	)
 	(no_connect
+		(at 173.99 120.65)
+	)
+	(no_connect
 		(at 137.16 135.89)
 	)
+	(no_connect
+		(at 173.99 130.81)
+	)
 	(wire
 		(pts
@@
 	(wire
 		(pts
-			(xy 233.68 151.13) (xy 243.84 151.13)
+			(xy 233.68 151.13) (xy 234.95 151.13)
 		)
 		(stroke
@@
 	(wire
 		(pts
+			(xy 234.95 151.13) (xy 243.84 151.13)
+		)
+		(stroke
+			(width 0)
+			(type default)
+		)
+	)
+	(wire
+		(pts
 			(xy 201.93 95.25) (xy 200.66 95.25)
 		)
@@
 			)
 		)
-		(property "Footprint" ""
+		(property "Footprint" "Resistor_SMD:R_0805_2012Metric"
 			(at 71.882 171.45 90)
 			(hide yes)
@@
 	)
 	(symbol
+		(lib_id "power:PWR_FLAG")
+		(at 234.95 151.13 0)
+		(unit 1)
+		(body_style 1)
+		(exclude_from_sim no)
+		(in_bom yes)
+		(on_board yes)
+		(in_pos_files yes)
+		(dnp no)
+		(fields_autoplaced yes)
+		(property "Reference" "#FLG01"
+			(at 234.95 149.225 0)
+			(hide yes)
+			(show_name no)
+			(do_not_autoplace no)
+			(effects
+				(font
+					(size 1.27 1.27)
+				)
+			)
+		)
+		(property "Value" "PWR_FLAG"
+			(at 234.95 146.05 0)
+			(show_name no)
+			(do_not_autoplace no)
+			(effects
+				(font
+					(size 1.27 1.27)
+				)
+			)
+		)
+		(property "Footprint" ""
+			(at 234.95 151.13 0)
+			(hide yes)
+			(show_name no)
+			(do_not_autoplace no)
+			(effects
+				(font
+					(size 1.27 1.27)
+				)
+			)
+		)
+		(property "Datasheet" ""
+			(at 234.95 151.13 0)
+			(hide yes)
+			(show_name no)
+			(do_not_autoplace no)
+			(effects
+				(font
+					(size 1.27 1.27)
+				)
+			)
+		)
+		(property "Description" "Special symbol for telling ERC where power comes from"
+			(at 234.95 151.13 0)
+			(hide yes)
+			(show_name no)
+			(do_not_autoplace no)
+			(effects
+				(font
+					(size 1.27 1.27)
+				)
+			)
+		)
+		(pin "1"
+		)
+		(instances
+			(project "variable load"
+				(path "/8b8c2ea1-e763-49aa-9f8d-d1a44d04f6ac"
+					(reference "#FLG01")
+					(unit 1)
+				)
+			)
+		)
+	)
+	(symbol
 		(lib_id "Isolator:6N137")
 		(at 57.15 175.26 0)
@@
 			)
 		)
-		(property "Footprint" ""
+		(property "Footprint" "Capacitor_SMD:C_0805_2012Metric"
 			(at 119.0752 180.34 0)
 			(hide yes)
@@
 			)
 		)
-		(property "Footprint" "R-78HE5.0-0.3:SIP900W75P254L1200H1300Q3"
+		(property "Footprint" "Package_SIP:SIP3_11.6x8.5mm"
 			(at 208.28 153.67 0)
 			(hide yes)
@@
 			)
 		)
-		(property "Footprint" "MCP4822-E_MS:SOP65P490X110-8N"
+		(property "Footprint" "Package_SO:MSOP-8_3x3mm_P0.65mm"
 			(at 119.38 138.43 0)
 			(hide yes)
@@
 			)
 		)
-		(property "Footprint" ""
+		(property "Footprint" "Capacitor_SMD:C_1206_3216Metric"
 			(at 225.7552 132.08 0)
 			(hide yes)
@@
 			)
 		)
-		(property "Footprint" ""
+		(property "Footprint" "Capacitor_SMD:C_0805_2012Metric"
 			(at 22.5552 142.24 0)
 			(hide yes)
@@
 			)
 		)
-		(property "Footprint" ""
+		(property "Footprint" "Resistor_SMD:R_0805_2012Metric"
 			(at 70.612 105.41 90)
 			(hide yes)
@@
 			)
 		)
-		(property "Footprint" ""
+		(property "Footprint" "Resistor_SMD:R_0805_2012Metric"
 			(at 140.462 138.43 90)
 			(hide yes)
@@
 			)
 		)
-		(property "Footprint" ""
+		(property "Footprint" "Resistor_SMD:R_0805_2012Metric"
 			(at 241.3 124.968 90)
 			(hide yes)
@@
 			)
 		)
-		(property "Footprint" ""
+		(property "Footprint" "Capacitor_SMD:C_0805_2012Metric"
 			(at 23.8252 110.49 0)
 			(hide yes)
@@
 			)
 		)
-		(property "Footprint" ""
+		(property "Footprint" "Capacitor_SMD:C_0805_2012Metric"
 			(at 22.5552 179.07 0)
 			(hide yes)
@@
 			)
 		)
-		(property "Footprint" ""
+		(property "Footprint" "Connector_PinHeader_2.54mm:PinHeader_1x04_P2.54mm_Vertical"
 			(at 158.75 173.99 0)
 			(hide yes)
@@
 			)
 		)
-		(property "Footprint" ""
+		(property "Footprint" "Capacitor_SMD:C_1206_3216Metric"
 			(at 129.2352 180.34 0)
 			(hide yes)
@@
 			)
 		)
-		(property "Footprint" ""
+		(property "Footprint" "Resistor_SMD:R_0805_2012Metric"
 			(at 71.882 138.43 90)
 			(hide yes)
@@
 			)
 		)
-		(property "Footprint" ""
+		(property "Footprint" "Resistor_SMD:R_0805_2012Metric"
 			(at 230.632 128.27 90)
 			(hide yes)
